File: voltage-regulator.kicad_pcb (KiCad board)
At the start: 2 copper layers, 32 parts, among them J1 PWR, J2 PWR, J3 PWR, U1 AMS1117-3.3, U2 TPS54302

Commit message: Added changes
Parts:
- removed TP1, TP5: GND_TP, Connector_Pin:Pin_D1.0mm_L10.0mm
- added H1: MountingHole, MountingHole:MountingHole_2.2mm_M2, F.Cu at (62.0, 26.0)
- added H2: MountingHole, MountingHole:MountingHole_2.2mm_M2, F.Cu at (41.8, 73.2)
- added H3: MountingHole, MountingHole:MountingHole_2.2mm_M2, F.Cu at (42.0, 26.0)
- added H4: MountingHole, MountingHole:MountingHole_2.2mm_M2, F.Cu at (62.2, 73.2)
- L1: footprint Inductor_SMD:L_0805_2012Metric -> SamacSys_Parts:INDPM6965X300N
- R2: footprint Resistor_SMD:R_0201_0603Metric -> Resistor_SMD:R_0402_1005Metric
- moved TP9 35.1 mm to (44.0, 54.5), turned to -90 degrees
- moved TP8 29.0 mm to (61.8, 57.8), turned to -90 degrees
- moved C9 19.3 mm to (57.0, 58.6)
- moved L1 13.4 mm to (51.9, 57.6), turned to 90 degrees
- moved R7 10.5 mm to (60.8, 62.0), turned to 180 degrees
- moved R5 10.5 mm to (58.2, 40.0), turned to -90 degrees
- moved R4 10.1 mm to (56.0, 63.9), turned to 0 degrees
- moved C5 10.1 mm to (48.1, 65.4)
- moved D3 9.92 mm to (60.4, 60.5)
- moved D1 8.28 mm to (60.5, 39.8)
- moved C8 7.00 mm to (55.5, 66.1), turned to 90 degrees
- moved C2 6.44 mm to (59.5, 31.1), turned to -90 degrees
- moved C6 5.88 mm to (49.8, 65.4), turned to 90 degrees
- moved R3 5.27 mm to (57.0, 66.1), turned to 90 degrees
- moved C7 4.76 mm to (53.1, 62.7), turned to 180 degrees
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Routing:
- net GND: track 22.0 -> 9.57 mm, vias 7 -> 47
- net +3.3V: track 16.0 -> 6.55 mm
- net /V_IN1: track 9.40 -> 0.00 mm
- net /VI: track 8.46 -> 0.00 mm
- net /SW: track 0.00 -> 6.03 mm
- net Net-(C8-Pad1): track 0.00 -> 5.37 mm
- net /FB: track 0.00 -> 5.31 mm
- net +5V: track 0.00 -> 2.85 mm
- net /BOOT: track 0.04 -> 1.67 mm
- net Net-(D3-K): track 0.00 -> 1.58 mm
- net Net-(D2-K): track 1.83 -> 3.27 mm
- added copper zone on F.Cu, net +5V
- added copper zone on F.Cu, net /VI
- added copper zone on F.Cu, net /VIN
- added copper zone on F.Cu, net /V_IN1
- added copper zone on B.Cu, net GND
Other:
- board outline added: 26 x 53 mm
- board text added: "12V In"
- board text added: "5V In 1A"
- board text added: "5V In 2A"
- board text added: "GND_TEST_P"
- board text added: "Quang D was here :))"
